File: High Voltage Bipolar Power Supply/FLYBACK_LT8304/FLYBACK_LT8304.kicad_sch (KiCad schematic)
At the start: 60 parts, among them J1 Conn_01x02, J2 Conn_01x03, Q1 Q_NPN_BCE, Q3 Q_PNP_BCE, T1 0399-T208, U1 LT8304, U2 LM317HV_TO-220, U3 LM337HV_TO220

Commit message: FLYBACK_LTC1624 : Schematic desing
Parts:
- removed C10, C11, C13, C15: 10u, symbol Device:C
- removed Q1: Q_NPN_BCE, symbol Device:Q_NPN_BCE
- removed Q3: Q_PNP_BCE, symbol Device:Q_PNP_BCE
- added C16, C2, C6, C8: 10u, Capacitor_SMD:C_2220_5750Metric_Pad1.97x5.40mm_HandSolder, symbol Device:C
- added HS1, HS2, HS3, HS4: TV5G, FLYBACK_LT8304:Heatsink_AAVID_TV5G_TO220_Horizontal, symbol Mechanical:Heatsink_Pad
- added Q1: TIP120, Package_TO_SOT_THT:TO-220-3_Horizontal_TabDown, symbol Transistor_BJT:TIP120
- added Q2: TIP125, Package_TO_SOT_THT:TO-220-3_Horizontal_TabDown, symbol Transistor_BJT:TIP125
- added TP4, TP5, TP6, TP7: TestPoint, TestPoint:TestPoint_THTPad_D3.0mm_Drill1.5mm, symbol Connector:TestPoint
- C1: renamed from C12; footprint (none) -> Capacitor_SMD:C_1206_3216Metric_Pad1.33x1.80mm_HandSolder
- C10: renamed from C16; footprint (none) -> Capacitor_SMD:C_1206_3216Metric_Pad1.33x1.80mm_HandSolder
- C11: renamed from C5; footprint (none) -> Capacitor_SMD:C_1812_4532Metric_Pad1.57x3.40mm_HandSolder; Package 1206 -> 1812; Voltage 200V -> 630V
- C12: renamed from C6; footprint (none) -> Capacitor_SMD:C_1812_4532Metric_Pad1.57x3.40mm_HandSolder; Package 1206 -> 1812; Voltage 200V -> 630V
- C13: renamed from C7; footprint (none) -> Capacitor_SMD:C_1812_4532Metric_Pad1.57x3.40mm_HandSolder
- C14, C17: footprint (none) -> Capacitor_SMD:C_2220_5750Metric_Pad1.97x5.40mm_HandSolder; Package 1206 -> 2220
- C15: renamed from C9; footprint (none) -> Capacitor_SMD:C_1206_3216Metric_Pad1.33x1.80mm_HandSolder
- C3: footprint (none) -> Capacitor_SMD:C_1210_3225Metric_Pad1.33x2.70mm_HandSolder
- C4: renamed from C2; footprint (none) -> Capacitor_SMD:C_1210_3225Metric_Pad1.33x2.70mm_HandSolder
- C5: renamed from C1; footprint (none) -> Capacitor_SMD:C_0805_2012Metric_Pad1.18x1.45mm_HandSolder; Package 1206 -> 0805; Voltage 25V -> 50V
- C7: renamed from C4; footprint (none) -> Capacitor_SMD:C_1206_3216Metric_Pad1.33x1.80mm_HandSolder
- C9: renamed from C8; footprint (none) -> Capacitor_SMD:C_0603_1608Metric_Pad1.08x0.95mm_HandSolder
- D1: renamed from D7; value D_Zener -> MMSZ5260BT1G; footprint (none) -> Diode_SMD:D_SOD-123
- D11: renamed from D5; footprint (none) -> LED_SMD:LED_0603_1608Metric_Pad1.05x0.95mm_HandSolder
- D12: renamed from D15; value D_Zener -> MMSZ5260BT1G; footprint (none) -> Diode_SMD:D_SOD-123
- D13: renamed from D16; value D_Zener -> BZT52C10-E3-08; footprint (none) -> Diode_SMD:D_SOD-123
- D14: renamed from D18; footprint (none) -> Diode_SMD:D_SMA
- D15: renamed from D17; footprint (none) -> Diode_SMD:D_SMA
- D16: renamed from D14; value D_Zener -> SMBJ5370B-TP; footprint (none) -> Diode_SMD:D_SMB
- D17: renamed from D12; footprint (none) -> Diode_SMD:D_SMA
- D18: renamed from D13; footprint (none) -> Diode_SMD:D_SMA
- D2: renamed from D8; value D_Zener -> BZT52C10-E3-08; footprint (none) -> Diode_SMD:D_SOD-123
- D3: renamed from D6; footprint (none) -> Diode_SMD:D_SMA
- D4: renamed from D9; value D_Zener -> SMBJ5370B-TP; footprint (none) -> Diode_SMD:D_SMB
- D5: renamed from D10; footprint (none) -> Diode_SMD:D_SMA
- D6: renamed from D11; footprint (none) -> Diode_SMD:D_SMA
- D7: renamed from D1; footprint (none) -> Diode_SMD:D_SOD-123F
- D8: renamed from D2; footprint (none) -> Diode_SMD:D_SOD-123F
- D9: renamed from D3; footprint (none) -> Diode_SMD:D_SOD-123F
- J1: value Conn_01x02 -> 1715721; footprint (none) -> TerminalBlock_Phoenix:TerminalBlock_Phoenix_MKDS-1,5-2_1x02_P5.00mm_Horizontal
- J2: value Conn_01x03 -> 1715734; footprint (none) -> TerminalBlock_Phoenix:TerminalBlock_Phoenix_MKDS-1,5-3-5.08_1x03_P5.08mm_Horizontal
- R1: renamed from R6; value 3k -> 3k/.25W; footprint (none) -> Resistor_SMD:R_0805_2012Metric_Pad1.20x1.40mm_HandSolder; Package 1206 -> 0805; Voltage 200V -> 100V
- R10: renamed from R9; footprint (none) -> Resistor_SMD:R_0805_2012Metric_Pad1.20x1.40mm_HandSolder
- R11: renamed from R10; footprint (none) -> Resistor_SMD:R_0805_2012Metric_Pad1.20x1.40mm_HandSolder
- R2: renamed from R8; footprint (none) -> Resistor_SMD:R_0805_2012Metric_Pad1.20x1.40mm_HandSolder
- R3: renamed from R7; footprint (none) -> Resistor_SMD:R_0805_2012Metric_Pad1.20x1.40mm_HandSolder
- R4: renamed from R2; footprint (none) -> Resistor_SMD:R_1206_3216Metric_Pad1.30x1.75mm_HandSolder
- R5: renamed from R4; footprint (none) -> Resistor_SMD:R_0603_1608Metric_Pad0.98x0.95mm_HandSolder
- R6: renamed from R1; footprint (none) -> Resistor_SMD:R_1206_3216Metric_Pad1.30x1.75mm_HandSolder
- R7: renamed from R3; footprint (none) -> Resistor_SMD:R_0603_1608Metric_Pad0.98x0.95mm_HandSolder
- R8: renamed from R11; value 3k -> 3k/.25W; footprint (none) -> Resistor_SMD:R_0805_2012Metric_Pad1.20x1.40mm_HandSolder; Package 1206 -> 0805; Voltage 200V -> 100V
- R9: renamed from R5; footprint (none) -> Resistor_SMD:R_0805_2012Metric_Pad1.20x1.40mm_HandSolder; Package 1206 -> 0805; Voltage 200V -> 100V
- TP1: renamed from TP3; footprint (none) -> TestPoint:TestPoint_THTPad_D3.0mm_Drill1.5mm
- TP2: renamed from TP1; footprint (none) -> TestPoint:TestPoint_THTPad_D3.0mm_Drill1.5mm
- TP3: renamed from TP2; footprint (none) -> TestPoint:TestPoint_THTPad_D3.0mm_Drill1.5mm
- TP8: renamed from TP4; footprint (none) -> TestPoint:TestPoint_THTPad_D3.0mm_Drill1.5mm
- U1: renamed from U2; footprint Package_TO_SOT_THT:TO-220-3_Vertical -> Package_TO_SOT_THT:TO-220-3_Horizontal_TabDown
- U3: footprint Package_TO_SOT_THT:TO-220-3_Vertical -> Package_TO_SOT_THT:TO-220-3_Horizontal_TabDown
- renumbered D4 to D10, U1 to U2
Connections:
- net +48V: now also C8.1
- net +HVDC: now also Q1.2 (C)
- net -48V: now also C17.2
- net -HVDC: now also Q2.2 (C)
- net GND1: now also C14.2, C17.1, C16.1, C2.2, C6.2, C8.2, TP4.1, TP5.1, TP6.1, TP7.1; no longer C14.1, C17.2
- net at D17.1 (K), R10.2, R11.1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: now also C16.2; no longer C14.2
- net at TH2.2, U3.2 (VI): now also Q2.3 (E)
- net at D5.2 (A), R2.1, R3.2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: now also C6.1
- net at D1.1 (K), R1.2: now also C2.1, Q1.1 (B)
- net at TH1.2, U1.3 (VI): now also Q1.3 (E)
- net at D12.2 (A), R8.2: now also C14.1, Q2.1 (B); no longer C17.1
- no-connect marks 0 -> 4
Other:
- note added: "Cap 10u/100V - 22201C106KAT2A Cap 10u/50V - UMJ325KB7106KMHP"
- moved on the sheet: C10, D12, D13, D14, D15, D16, D17, D18, D4, R10, R11, R8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
