File: High Voltage Bipolar Power Supply/FLYBACK_LTC1624/FLYBACK_LTC1624.kicad_pcb (KiCad board)
At the start: 2 copper layers, 0 parts

Commit message: FLYBACK_LTC1624: PCB layout
Parts:
- added C1: 0.01u, Capacitor_SMD:C_0603_1608Metric_Pad1.08x0.95mm_HandSolder, F.Cu at (117.5, 101.3)
- added C10: 10u, Capacitor_SMD:C_1206_3216Metric_Pad1.33x1.80mm_HandSolder, F.Cu at (135.6, 115.4)
- added C11: 0.1u, Capacitor_SMD:C_0603_1608Metric_Pad1.08x0.95mm_HandSolder, F.Cu at (131.2, 112.4)
- added C12: 0.1u, Capacitor_SMD:C_0603_1608Metric_Pad1.08x0.95mm_HandSolder, F.Cu at (147.8, 112.4)
- added C13: 10u, Capacitor_SMD:C_1206_3216Metric_Pad1.33x1.80mm_HandSolder, F.Cu at (144.3, 115.6)
- added C14: 0.22u, Capacitor_SMD:C_1206_3216Metric_Pad1.33x1.80mm_HandSolder, F.Cu at (166.9, 92.8)
- added C15: 1u, Capacitor_SMD:C_1206_3216Metric_Pad1.33x1.80mm_HandSolder, F.Cu at (162.8, 101.6)
- added C16: 1u, Capacitor_SMD:C_1206_3216Metric_Pad1.33x1.80mm_HandSolder, F.Cu at (162.8, 78.7)
- added C17: 0.05u, Capacitor_SMD:C_1206_3216Metric_Pad1.33x1.80mm_HandSolder, F.Cu at (173.9, 74.3)
- added C18: 0.05u, Capacitor_SMD:C_1206_3216Metric_Pad1.33x1.80mm_HandSolder, F.Cu at (162.8, 124.7)
- added C19: 10u, FLYBACK_LTC1624:C_2220_5750Metric_Pad1.97x5.40mm_HandSolder, F.Cu at (190.6, 76.7)
- added C2: 330u, Capacitor_SMD:CP_Elec_10x10, F.Cu at (108.2, 89.3)
- added C20: 10u, FLYBACK_LTC1624:C_2220_5750Metric_Pad1.97x5.40mm_HandSolder, F.Cu at (157.1, 122.3)
- added C21: 10u, FLYBACK_LTC1624:C_2220_5750Metric_Pad1.97x5.40mm_HandSolder, F.Cu at (173.0, 107.1)
- added C22: 10u, FLYBACK_LTC1624:C_2220_5750Metric_Pad1.97x5.40mm_HandSolder, F.Cu at (195.2, 124.1)
- added C23: 10u, FLYBACK_LTC1624:C_2220_5750Metric_Pad1.97x5.40mm_HandSolder, F.Cu at (182.5, 107.1)
- added C24: 10u, FLYBACK_LTC1624:C_2220_5750Metric_Pad1.97x5.40mm_HandSolder, F.Cu at (195.2, 114.8)
- added C3: 1u, Capacitor_SMD:C_0603_1608Metric_Pad1.08x0.95mm_HandSolder, F.Cu at (121.5, 98.2)
- added C4: 10u, Capacitor_SMD:C_1210_3225Metric_Pad1.33x2.70mm_HandSolder, F.Cu at (116.7, 112.4)
- added C5: 1u, Capacitor_SMD:C_1206_3216Metric_Pad1.33x1.80mm_HandSolder, F.Cu at (115.6, 92.5)
- added C6: 10u, Capacitor_SMD:C_1210_3225Metric_Pad1.33x2.70mm_HandSolder, F.Cu at (125.6, 112.4)
- added C7: 1u, Capacitor_SMD:C_0603_1608Metric_Pad1.08x0.95mm_HandSolder, F.Cu at (117.5, 87.5)
- added C8: 10u, Capacitor_SMD:C_1206_3216Metric_Pad1.33x1.80mm_HandSolder, F.Cu at (129.3, 122.4)
- added C9: 0.22u, Capacitor_SMD:C_1206_3216Metric_Pad1.33x1.80mm_HandSolder, F.Cu at (133.3, 83.2)
- added D1: MURS120T3, Diode_SMD:D_SMB, F.Cu at (161.5, 94.4)
- added D10: MRA4003T3G, Diode_SMD:D_SMA, F.Cu at (173.7, 87.5)
- added D11: MRA4003T3G, Diode_SMD:D_SMA, F.Cu at (175.8, 123.7)
- added D12: MRA4003T3G, Diode_SMD:D_SMA, F.Cu at (182.1, 101.5)
- added D13: MRA4003T3G, Diode_SMD:D_SMA, F.Cu at (189.6, 115.2)
- added D2: MURS120T3, Diode_SMD:D_SMB, F.Cu at (161.5, 86.1)
- added D3: MMSZ5260BT1G, Diode_SMD:D_SOD-123, F.Cu at (188.1, 82.7)
- added D4: BZT52C10-E3-08, Diode_SMD:D_SOD-123, F.Cu at (193.2, 82.7)
- added D5: MMSZ5260BT1G, Diode_SMD:D_SOD-123, F.Cu at (161.4, 116.4)
- added D6: BZT52C10-E3-08, Diode_SMD:D_SOD-123, F.Cu at (161.4, 113.7)
- added D7: MRA4003T3G, Diode_SMD:D_SMA, F.Cu at (181.4, 87.5)
- added D8: MRA4003T3G, Diode_SMD:D_SMA, F.Cu at (197.9, 77.3)
- added D9: MRA4003T3G, Diode_SMD:D_SMA, F.Cu at (175.8, 116.2)
- added HS1: HS-S01, FLYBACK_LTC1624:Heatsink_Stonecold_HS-S01_13.21x6.35mm, F.Cu at (179.6, 119.9)
- added HS2: HS-S01, FLYBACK_LTC1624:Heatsink_Stonecold_HS-S01_13.21x6.35mm, F.Cu at (177.5, 83.6)
- added HS3: HS-S01, FLYBACK_LTC1624:Heatsink_Stonecold_HS-S01_13.21x6.35mm, F.Cu at (171.9, 119.9)
- added HS4: HS-S01, FLYBACK_LTC1624:Heatsink_Stonecold_HS-S01_13.21x6.35mm, F.Cu at (177.5, 91.5)
- added J1: 1715721, TerminalBlock_Phoenix:TerminalBlock_Phoenix_MKDS-1,5-2_1x02_P5.00mm_Horizontal, F.Cu at (107.3, 100.2)
- added J2: Conn_01x02, Connector_PinHeader_2.54mm:PinHeader_1x02_P2.54mm_Vertical, F.Cu at (138.3, 127.4)
- added J3: 1715734, TerminalBlock_Phoenix:TerminalBlock_Phoenix_MKDS-1,5-3-5.08_1x03_P5.08mm_Horizontal, F.Cu at (196.6, 101.0)
- added L1: TCK-141, FLYBACK_LTC1624:TCK-141, F.Cu at (121.2, 112.4)
- added Q1: PZT2222A, Package_TO_SOT_SMD:SOT-223-3_TabPin2, F.Cu at (119.5, 81.2)
- added Q2: IRL540NS, Package_TO_SOT_SMD:TO-263-2, F.Cu at (130.4, 97.6)
- added Q3: TIP125, Package_TO_SOT_THT:TO-220-3_Vertical, F.Cu at (180.1, 78.7)
- added Q4: TIP120, Package_TO_SOT_THT:TO-220-3_Vertical, F.Cu at (167.0, 117.5)
- added R1: 1k, Resistor_SMD:R_0603_1608Metric_Pad0.98x0.95mm_HandSolder, F.Cu at (117.5, 98.2)
- added R10: 15k, Resistor_SMD:R_0603_1608Metric_Pad0.98x0.95mm_HandSolder, F.Cu at (147.3, 109.5)
- added R11: 18k, Resistor_SMD:R_1206_3216Metric_Pad1.30x1.75mm_HandSolder, F.Cu at (160.3, 101.6)
- added R12: 18k, Resistor_SMD:R_1206_3216Metric_Pad1.30x1.75mm_HandSolder, F.Cu at (160.3, 78.7)
- added R13: 47, Resistor_SMD:R_1206_3216Metric_Pad1.30x1.75mm_HandSolder, F.Cu at (166.9, 98.0)
- added R14: 620k, Resistor_SMD:R_1206_3216Metric_Pad1.30x1.75mm_HandSolder, F.Cu at (153.0, 110.7)
- added R15: 3k/.25W, Resistor_SMD:R_0805_2012Metric_Pad1.20x1.40mm_HandSolder, F.Cu at (178.8, 74.3)
- added R16: 3k/.25W, Resistor_SMD:R_0805_2012Metric_Pad1.20x1.40mm_HandSolder, F.Cu at (162.8, 119.9)
- added R17: 5k11/0.5W, Resistor_SMD:R_0805_2012Metric_Pad1.20x1.40mm_HandSolder, F.Cu at (172.3, 101.5)
- added R18: 5k11/0.5W, Resistor_SMD:R_0805_2012Metric_Pad1.20x1.40mm_HandSolder, F.Cu at (189.6, 125.2)
- added R19: 150/.25W, Resistor_SMD:R_0805_2012Metric_Pad1.20x1.40mm_HandSolder, F.Cu at (176.4, 101.5)
- added R2: CRF1206-FZ-R020ELF, Resistor_SMD:R_1206_3216Metric_Pad1.30x1.75mm_HandSolder, F.Cu at (119.5, 75.7)
- added R20: 150/.25W, Resistor_SMD:R_0805_2012Metric_Pad1.20x1.40mm_HandSolder, F.Cu at (189.6, 120.9)
- added R3: 220, Resistor_SMD:R_1206_3216Metric_Pad1.30x1.75mm_HandSolder, F.Cu at (127.4, 83.2)
- added R4: 43k, Resistor_SMD:R_1206_3216Metric_Pad1.30x1.75mm_HandSolder, F.Cu at (127.4, 78.9)
- added R5: 10, Resistor_SMD:R_0603_1608Metric_Pad0.98x0.95mm_HandSolder, F.Cu at (121.5, 87.5)
- added R6: 15k, Resistor_SMD:R_0603_1608Metric_Pad0.98x0.95mm_HandSolder, F.Cu at (121.5, 101.3)
- added R7: 100, Resistor_SMD:R_0603_1608Metric_Pad0.98x0.95mm_HandSolder, F.Cu at (121.5, 104.3)
- added R8: 47, Resistor_SMD:R_1206_3216Metric_Pad1.30x1.75mm_HandSolder, F.Cu at (133.3, 78.9)
- added R9: 620k, Resistor_SMD:R_1206_3216Metric_Pad1.30x1.75mm_HandSolder, F.Cu at (153.0, 106.9)
- added REF**: Symbol_HighVoltage_Triangle_6x6mm_Copper, Symbol:Symbol_HighVoltage_Triangle_6x6mm_Copper, F.Cu at (106.0, 125.5)
- added T1: VP3-0138, FLYBACK_LTC1624:VP3, F.Cu at (147.1, 88.6)
- added TP1: TestPoint, TestPoint:TestPoint_THTPad_D3.0mm_Drill1.5mm, F.Cu at (161.0, 108.6)
- added TP2: TestPoint, TestPoint:TestPoint_THTPad_D3.0mm_Drill1.5mm, F.Cu at (166.1, 108.6)
- added TP3: TestPoint, TestPoint:TestPoint_THTPad_D3.0mm_Drill1.5mm, F.Cu at (166.5, 73.7)
- added TP4: TestPoint, TestPoint:TestPoint_THTPad_D3.0mm_Drill1.5mm, F.Cu at (161.4, 73.7)
- added U1: LTC1624CS8, Package_SO:SOIC-8_3.9x4.9mm_P1.27mm, F.Cu at (119.8, 92.6)
- added U2: TSR_1-2450, Converter_DCDC:Converter_DCDC_TRACO_TSR-1_THT, F.Cu at (118.6, 122.6)
- added U3: ADUM4195-1, Package_SO:SSO-8_6.8x5.9mm_P1.27mm_Clearance8mm, F.Cu at (139.6, 110.5)
- added U4: TBA1-0511E, Converter_DCDC:Converter_DCDC_TRACO_TBA1-xxxxE_Single_THT, F.Cu at (134.4, 119.9)
- added U5: LM337HV_TO220, Package_TO_SOT_THT:TO-220-3_Vertical, F.Cu at (175.0, 96.4)
- added U6: LM317HV_TO-220, Package_TO_SOT_THT:TO-220-3_Vertical, F.Cu at (184.5, 122.4)
Other:
- board outline added: 100 x 60 mm
- board text added: "+50V"
- board text added: "+HV"
- board text added: "-50V"
- board text added: "-HV"
- board text added: "24V DC"
- board text added: "GND"
